File: tests/data/layout1.kicad_pcb (KiCad board)
At the start: 2 copper layers, 38 x 14 mm, 28 parts, among them J1 MICRO-USB-B-alt, P1 CONN_01X06, U1 FTDI-FT230X, U2 MCP1703-alt

Commit message: deal with kicad quoting in layout files
Other:
- board text added: "25" (quote test!)"
Changed lines of the file:
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@@
     (area 156.2 52.3 224.448402 96.800001)
     (thickness 1.6)
-    (drawings 23)
+    (drawings 24)
     (tracks 193)
     (zones 0)
@@
       (net 25 "Net-(D4-Pad2)"))
   )
+  (gr_text "25\" (quote test!)" (at 200.6 49.3) (layer Eco2.User)
+    (effects (font (size 1.5 1.5) (thickness 0.3)))
+  )
   (gr_text OFF (at 205 69) (layer B.SilkS)
