File: tests/data/schematic1.sch (KiCad schematic (older format))
At the start: 26 parts, among them J1 USB-C-WE-623723x00011, P1 CONN_01X12, P2 CONN_01X12, P3 CONN_02X03, U1 EFM32HG310, U2 MCP1703-alt, U3 ST-USBLC6-2, X1 32kHz/9pF, X2 24MHz/9pF

Commit message: add text examples
Connections:
- net labels added: GLOBALDOWN, GLOBALRIGHT, GLOBALUP, IAMGLOBAL, IAMHIERARCHICAL
Other:
- note added: "IAMANOTE"
Changed lines of the file:
@@
 EESchema Schematic File Version 2
-LIBS:power
-LIBS:conn
-EELAYER 26 0
+LIBS:schematic1-cache
+EELAYER 25 0
 EELAYER END
 $Descr A4 11693 8268
@@
 Text Label 7050 3200 0    60   ~ 0
 D-2
+Text GLabel 8175 1650 0    60   Input ~ 0
+IAMGLOBAL
+Text HLabel 9200 1650 0    60   Input ~ 0
+IAMHIERARCHICAL
+Text GLabel 8175 1875 2    60   Input ~ 0
+GLOBALRIGHT
+Text GLabel 7775 2400 1    60   Input ~ 0
+GLOBALUP
+Text GLabel 8050 2050 3    60   Input ~ 0
+GLOBALDOWN
+Text Notes 8025 5400 0    60   ~ 0
+IAMANOTE
 $EndSCHEMATC

Commit message: text-type parsing and generation for schematic (unused yet)
Connections:
- net labels added: IAMBOLD, IAMBOLDITALIC, IAMITALIC
Changed lines of the file:
@@
 EESchema Schematic File Version 2
-LIBS:schematic1-cache
 EELAYER 25 0
 EELAYER END
@@
 Text Notes 8025 5400 0    60   ~ 0
 IAMANOTE
+Text Label 8800 2175 0    60   Italic 0
+IAMITALIC
+Text Label 8800 2350 0    60   ~ 12
+IAMBOLD
+Text Label 9300 2175 0    60   Italic 12
+IAMBOLDITALIC
 $EndSCHEMATC
